File: universal-home-esp-module/universal-home-esp-module.kicad_pcb (KiCad board)
At the start: 2 copper layers, 51.7 x 46 mm, 12 parts, among them J1 ES8311 CODEC, J10 ESP32_RPINS, J2 LDR MOD, J3 RELAYS, J4 RGB LED, J5 ENV SENSOR, J6 5V PWR, J7 EXT_GPIO, J8 EXT_I2C, J9 ESP32_LPINS, U1 ESP32-C3_SUPERMINI_SMD, U2 74HC595

Commit message: update schematic
Parts:
- J10, J9: footprint Connector_PinSocket_2.54mm:PinSocket_1x08_P2.54mm_Vertical -> Connector_PinHeader_2.54mm:PinHeader_1x08_P2.54mm_Vertical
- J2: footprint Connector_PinSocket_2.54mm:PinSocket_1x03_P2.54mm_Vertical -> Connector_PinHeader_2.54mm:PinHeader_1x03_P2.54mm_Vertical
- J3: footprint Connector_PinSocket_2.54mm:PinSocket_1x06_P2.54mm_Vertical -> Connector_PinHeader_2.54mm:PinHeader_1x06_P2.54mm_Vertical
- moved J7 8.05 mm to (69.3, 76.2)
- moved J2 8.05 mm to (97.5, 70.8)
- moved J5 8.05 mm to (69.3, 70.6)
- moved J6 8.05 mm to (83.2, 79.7)
- moved U2 8.05 mm to (63.4, 45.9)
- moved J10 8.05 mm to (102.1, 45.0)
- moved U1 8.05 mm to (89.6, 54.9)
- moved J1 8.05 mm to (107.6, 44.9)
- moved J3 8.05 mm to (64.2, 81.7)
- moved J4 8.05 mm to (97.5, 79.6)
- moved J8 8.05 mm to (83.3, 70.8)
- moved J9 8.05 mm to (77.0, 45.0)
Connections:
- J3 pad 1: 3V3 -> 5V
- U2 pad 10: unconnected-(U2-~{SRCLR}-Pad10) -> 5V
- U2 pad 13: unconnected-(U2-~{OE}-Pad13) -> GND
Routing:
- net 5V: track 74.6 -> 119.6 mm
- net 3V3: track 112.6 -> 98.2 mm
- net GND: vias 123 -> 127
- net Net-(J3-Pin_4): vias 4 -> 0
- net Net-(J3-Pin_5): vias 7 -> 2
